Commit message: debug loading issue in rviz

File: isaac_sim_test/gcr16_2000/v1/urdf/gcr16_common.xacro (robot description, xacro)
@@ -16,5 +16,5 @@
         <origin xyz="0 0 0" rpy="0 0 0"/>
         <geometry>
-          <mesh filename="file://${mesh_dir}/${stl_name}" scale="0.001 0.001 0.001"/>
+          <mesh filename="package://gcr16_2000_v1/meshes/${stl_name}" scale="0.001 0.001 0.001"/>
         </geometry>
       </xacro:if>
@@ -33,5 +33,5 @@
       <xacro:if value="${use_cad_meshes}">
         <geometry>
-          <mesh filename="file://${mesh_dir}/${stl_name}" scale="0.001 0.001 0.001"/>
+          <mesh filename="package://gcr16_2000_v1/meshes/${stl_name}" scale="0.001 0.001 0.001"/>
         </geometry>
       </xacro:if>
